File: LEDs1.sch (KiCad schematic (older format))
At the start: 86 parts, among them Q1 Q_NMOS_GSD

Commit message: Schematic is almost finished. The MCLR circuit needs completing, the hour/minute inputs also need their input protection.
After that, I might have one of the guys from work review it. But, who knows.
Parts:
- gave numbers to parts that had none: 77
