File: PowerMicroRTCandComm.sch (KiCad schematic (older format))
At the start: 31 parts, among them J1 USB_C_Receptacle_USB2.0, U1 NUP2202, U2 PIC18LF46K80-IPT, U3 LM1117-3.3, U4 DS3231MZ, U5 FT230XS

Commit message: Schematic is almost finished. The MCLR circuit needs completing, the hour/minute inputs also need their input protection.
After that, I might have one of the guys from work review it. But, who knows.
Connections:
- net NINE_H: now reaches U2.10 (CANTX/CTED1/INT2/RB2)
- net TEN_H: now reaches U2.11 (CANRX/CTED2/INT3/RB3)
- net TEN_H: now also U2.32 (RC0/SOSCO/SCLKI)
- net ONE_H: now reaches U2.14 (AN9/CTPLS/KBI0/RB4)
- net POT_IN: now reaches U2.19 (CVref/AN0/ULPWU/RA0)
- net ELEVEN_H: now reaches U2.2 (RD4/ECCP1/P1A/PSP4)
- net IT_IS: now reaches U2.20 (AN1/C1INC/RA1)
- net HALF: now reaches U2.21 (VREF-/AN2/C2INC/RA2)
- net FIVE_M: now reaches U2.22 (Vref+/AN3/RA3)
- net PAST: now reaches U2.24 (AN4/HLVDIN/T1CKI/~SS~/RA5)
- net SIX_H: now reaches U2.25 (RE0/AN5/~RD~)
- net FOUR_H: now reaches U2.26 (RE1/AN6/C1OUT/~WR~)
- net FIVE_H: now reaches U2.27 (RE2/AN7/C2OUT/~CS~)
- net TWELVE: now reaches U2.3 (RD5/P1B/PSP5)
- net TO: now reaches U2.35 (RC1/SOSCI)
- net THREE_H: now reaches U2.36 (RC2/T1G/CCP2)
- net EIGHT_H: now reaches U2.38 (RD0/C1INA/PSP0)
- net QUARTER: now reaches U2.39 (RD1/C1INB/PSP1)
- net OCLOCK: now reaches U2.4 (RD6/TX2/CK2/P1C/PSP6)
- net MINUTES: now reaches U2.40 (RD2/C2INA/PSP2)
- net TWENTY_M: now reaches U2.41 (RD3/C2INB/CTMUI/PSP3)
- net SEVEN_H: now reaches U2.43 (RC5/SDO)
- net TWO_H: now reaches U2.5 (RD7/RX2/DT2/P1D/PSP7)
- net HOUR_ADJUST: now reaches U2.8 (AN10/FLT0/INT0/RB0)
- net MINUTE_ADJUST: now reaches U2.9 (AN8/CTDIN/INT1/RB1)
- no-connect marks 8 -> 15
Changed lines of the file:
@@
 Wire Wire Line
 	3750 3650 3750 3600
-Text Label 2000 5700 0    50   ~ 0
+Text Label 1800 5700 0    50   ~ 0
 SDA
-Text Label 2000 5600 0    50   ~ 0
+Text Label 1800 5600 0    50   ~ 0
 SCL
-Wire Wire Line
-	2350 5700 2000 5700
-Wire Wire Line
-	2350 5600 2000 5600
 Text Label 1800 5900 0    50   ~ 0
 UART_TX
@@
 NoConn ~ 1600 2400
 NoConn ~ 1600 2300
+Text Label 5450 4800 0    50   ~ 0
+IT_IS
+Text Label 5450 4900 0    50   ~ 0
+HALF
+Text Label 5450 5000 0    50   ~ 0
+FIVE_M
+Text Label 5450 5100 0    50   ~ 0
+PAST
+Text Label 1800 4100 0    50   ~ 0
+FOUR_H
+Text Label 1800 4200 0    50   ~ 0
+FIVE_H
+Text Label 5450 5500 0    50   ~ 0
+NINE_H
+Text Label 5450 5600 0    50   ~ 0
+TEN_H
+Text Label 5450 5700 0    50   ~ 0
+ONE_H
+Text Label 1800 5100 0    50   ~ 0
+TWO_H
+Text Label 1800 4000 0    50   ~ 0
+SIX_H
+Text Label 1800 5300 0    50   ~ 0
+TEN_H
+Text Label 1800 5400 0    50   ~ 0
+TO
+Text Label 1800 5500 0    50   ~ 0
+THREE_H
+Text Label 1800 5800 0    50   ~ 0
+SEVEN_H
+Text Label 1800 4400 0    50   ~ 0
+EIGHT_H
+Text Label 1800 4500 0    50   ~ 0
+QUARTER
+Text Label 1800 4600 0    50   ~ 0
+MINUTES
+Text Label 1800 4700 0    50   ~ 0
+TWENTY_M
+Text Label 1800 4800 0    50   ~ 0
+ELEVEN_H
+Text Label 1800 4900 0    50   ~ 0
+TWELVE
+Text Label 1800 5000 0    50   ~ 0
+OCLOCK
+Wire Wire Line
+	1800 5600 2350 5600
+Wire Wire Line
+	1800 5700 2350 5700
+Wire Wire Line
+	2350 5800 1800 5800
+Wire Wire Line
+	2350 5500 1800 5500
+Wire Wire Line
+	1800 5400 2350 5400
+Wire Wire Line
+	2350 5300 1800 5300
+Wire Wire Line
+	1800 5100 2350 5100
+Wire Wire Line
+	1800 5000 2350 5000
+Wire Wire Line
+	1800 4900 2350 4900
+Wire Wire Line
+	1800 4800 2350 4800
+Wire Wire Line
+	1800 4700 2350 4700
+Wire Wire Line
+	1800 4600 2350 4600
+Wire Wire Line
+	1800 4500 2350 4500
+Wire Wire Line
+	1800 4400 2350 4400
+Wire Wire Line
+	1800 4200 2350 4200
+Wire Wire Line
+	1800 4100 2350 4100
+Wire Wire Line
+	1800 4000 2350 4000
+Wire Wire Line
+	5150 4800 5450 4800
+Wire Wire Line
+	5150 4900 5450 4900
+Wire Wire Line
+	5150 5000 5450 5000
+Wire Wire Line
+	5150 5100 5450 5100
+Wire Wire Line
+	5150 5500 5450 5500
+Wire Wire Line
+	5150 5600 5450 5600
+Wire Wire Line
+	5150 5700 5450 5700
+NoConn ~ 5150 5800
+NoConn ~ 3150 6500
+NoConn ~ 3050 6500
+NoConn ~ 2950 6500
+NoConn ~ 2850 6500
+NoConn ~ 5150 4200
+NoConn ~ 5150 4300
+Text Label 5450 4700 0    50   ~ 0
+POT_IN
+Wire Wire Line
+	5150 4700 5450 4700
+Text Label 5450 5300 0    50   ~ 0
+HOUR_ADJUST
+Text Label 5450 5400 0    50   ~ 0
+MINUTE_ADJUST
+Wire Wire Line
+	5450 5400 5150 5400
+Wire Wire Line
+	5150 5300 5450 5300
 $EndSCHEMATC
